File: Apple/Apple IIGS/IIgs/ROM3 Schematic/IWM-4.sch (KiCad schematic (older format))
At the start: 77 parts, among them J15 Conn_01x11, J16 Conn_01x11, J8 Conn_01x21, J9 Game Port, U13 74LS51, Y2 3.6864 MHz

Commit message: added more notes on keyboard page. refined some hierarchical labels.
Other:
- moved on the sheet: C34, C35
Changed lines of the file:
@@
 Wire Wire Line
 	5200 10550 5300 10550
-Text Notes 1800 9100 0    50   ~ 0
+Text Notes 2350 9100 0    50   ~ 0
 Should SW1/SW2 be heirarchical?
 Connection ~ 1050 10300
@@
 Text Label 1400 9300 2    50   ~ 0
 SW1-CAPL
-Text Label 1900 9450 0    50   ~ 0
+Text Label 2450 9450 0    50   ~ 0
 SW0-OAPL
-Text Label 1900 9300 0    50   ~ 0
+Text Label 2450 9300 0    50   ~ 0
 SW1-CAPL
 $Comp
 L Device:C_Small C34
 U 1 1 5F144A5D
-P 2400 9550
-F 0 "C34" H 2492 9596 50  0000 L CNN
-F 1 "0.01u" H 2492 9505 50  0000 L CNN
-F 2 "" H 2400 9550 50  0001 C CNN
-F 3 "~" H 2400 9550 50  0001 C CNN
-	1    2400 9550
+P 2950 9550
+F 0 "C34" H 3042 9596 50  0000 L CNN
+F 1 "0.01u" H 3042 9505 50  0000 L CNN
+F 2 "" H 2950 9550 50  0001 C CNN
+F 3 "~" H 2950 9550 50  0001 C CNN
+	1    2950 9550
 	1    0    0    -1
 $EndComp
@@
 L Device:C_Small C35
 U 1 1 5F144E19
-P 2800 9550
-F 0 "C35" H 2892 9596 50  0000 L CNN
-F 1 ".01u" H 2892 9505 50  0000 L CNN
-F 2 "" H 2800 9550 50  0001 C CNN
-F 3 "~" H 2800 9550 50  0001 C CNN
-	1    2800 9550
+P 3350 9550
+F 0 "C35" H 3442 9596 50  0000 L CNN
+F 1 ".01u" H 3442 9505 50  0000 L CNN
+F 2 "" H 3350 9550 50  0001 C CNN
+F 3 "~" H 3350 9550 50  0001 C CNN
+	1    3350 9550
 	1    0    0    -1
 $EndComp
 Wire Wire Line
-	2400 9650 2400 9750
+	2950 9650 2950 9750
 Wire Wire Line
-	2400 9750 2600 9750
+	2950 9750 3150 9750
 Wire Wire Line
-	2800 9750 2800 9650
+	3350 9750 3350 9650
 Wire Wire Line
-	2400 9450 1900 9450
-Wire Wire Line
-	2800 9300 2800 9450
+	3350 9300 3350 9450
 $Comp
 L power:GNDPWR #PWR?
 U 1 1 5F183B1D
-P 2600 9750
-F 0 "#PWR?" H 2600 9550 50  0001 C CNN
-F 1 "GNDPWR" H 2604 9596 50  0001 C CNN
-F 2 "" H 2600 9700 50  0001 C CNN
-F 3 "" H 2600 9700 50  0001 C CNN
-	1    2600 9750
+P 3150 9750
+F 0 "#PWR?" H 3150 9550 50  0001 C CNN
+F 1 "GNDPWR" H 3154 9596 50  0001 C CNN
+F 2 "" H 3150 9700 50  0001 C CNN
+F 3 "" H 3150 9700 50  0001 C CNN
+	1    3150 9750
 	1    0    0    -1
 $EndComp
-Connection ~ 2600 9750
+Connection ~ 3150 9750
 Wire Wire Line
-	2600 9750 2800 9750
-Wire Wire Line
-	1900 9300 2800 9300
+	3150 9750 3350 9750
 Text Notes 2100 10200 0    50   ~ 0
 C34 & C35\nOptional \nFor Impoved EMI
+Text HLabel 2400 9300 0    50   Input ~ 0
+SW1-CAPL
+Text HLabel 2400 9450 0    50   Input ~ 0
+SW0-OAPL
+Wire Wire Line
+	2400 9300 3350 9300
+Wire Wire Line
+	2400 9450 2950 9450
 $EndSCHEMATC

Commit message: continued refinements
Changed lines of the file:
@@
 $Descr A3 16535 11693
 encoding utf-8
-Sheet 4 10
+Sheet 1 1
 Title "IWM, Serial, Gameport"
 Date ""
@@
 Wire Wire Line
 	2650 3050 3000 3050
-Text GLabel 1100 3200 0    50   Input ~ 0
-INTDEV6.L
 Text Label 1600 3200 2    50   ~ 0
 INTDEV6.L
@@
 Text HLabel 1200 2750 0    50   Input ~ 0
 7M.H
-Text Label 1450 2950 2    50   ~ 0
+Text Label 1600 2950 2    50   ~ 0
 Q3.H
 Wire Wire Line
@@
 Wire Wire Line
 	2400 9450 2950 9450
+Text HLabel 1100 3200 0    50   Input ~ 0
+INTDEV6.L
 $EndSCHEMATC

Commit message: continued fixes while working on golden delicious project
Other:
- moved on the sheet: R120, R190, TP111, TP153
Changed lines of the file:
@@
 $Descr A3 16535 11693
 encoding utf-8
-Sheet 1 1
+Sheet 4 10
 Title "IWM, Serial, Gameport"
 Date ""
@@
 L Device:R_Small R120
 U 1 1 5EA01B07
-P 1950 1050
-F 0 "R120" V 1850 1050 50  0000 C CNN
-F 1 "470" V 2050 1050 50  0000 C CNN
-F 2 "" H 1950 1050 50  0001 C CNN
-F 3 "~" H 1950 1050 50  0001 C CNN
-	1    1950 1050
+P 7950 850
+F 0 "R120" V 7850 850 50  0000 C CNN
+F 1 "470" V 8050 850 50  0000 C CNN
+F 2 "" H 7950 850 50  0001 C CNN
+F 3 "~" H 7950 850 50  0001 C CNN
+	1    7950 850
 	0    1    1    0
 $EndComp
 Wire Wire Line
-	1850 1050 1700 1050
-Text Label 1600 1050 2    50   ~ 0
+	7850 850  7700 850
+Text Label 7600 850  2    50   ~ 0
 3.5DIK
 $Comp
 L Connector:TestPoint TP111
 U 1 1 5EA09332
-P 1700 850
-F 0 "TP111" H 1758 922 50  0000 L CNN
-F 1 "TestPoint" H 1758 877 50  0001 L CNN
-F 2 "" H 1900 850 50  0001 C CNN
-F 3 "~" H 1900 850 50  0001 C CNN
-	1    1700 850
-	1    0    0    -1
-$EndComp
-Wire Wire Line
-	1700 850  1700 1050
-Connection ~ 1700 1050
-Wire Wire Line
-	1700 1050 1150 1050
+P 7700 650
+F 0 "TP111" H 7758 722 50  0000 L CNN
+F 1 "TestPoint" H 7758 677 50  0001 L CNN
+F 2 "" H 7900 650 50  0001 C CNN
+F 3 "~" H 7900 650 50  0001 C CNN
+	1    7700 650
+	1    0    0    -1
+$EndComp
+Wire Wire Line
+	7700 650  7700 850
+Connection ~ 7700 850
+Wire Wire Line
+	7700 850  7150 850
 Wire Wire Line
 	2650 3050 3000 3050
@@
 L Connector:TestPoint TP153
 U 1 1 5EA47314
-P 1550 1600
-F 0 "TP153" V 1653 1672 50  0000 C CNN
-F 1 "TestPoint" H 1608 1627 50  0001 L CNN
-F 2 "" H 1750 1600 50  0001 C CNN
-F 3 "~" H 1750 1600 50  0001 C CNN
-	1    1550 1600
+P 7550 1400
+F 0 "TP153" V 7653 1472 50  0000 C CNN
+F 1 "TestPoint" H 7608 1427 50  0001 L CNN
+F 2 "" H 7750 1400 50  0001 C CNN
+F 3 "~" H 7750 1400 50  0001 C CNN
+	1    7550 1400
 	0    -1   -1   0
 $EndComp
 Wire Wire Line
-	1550 1600 1700 1600
+	7550 1400 7700 1400
 $Comp
 L Device:R_Small R190
 U 1 1 5EA4A8B7
-P 1950 1400
-F 0 "R190" V 1850 1400 50  0000 C CNN
-F 1 "470" V 2050 1400 50  0000 C CNN
-F 2 "" H 1950 1400 50  0001 C CNN
-F 3 "~" H 1950 1400 50  0001 C CNN
-	1    1950 1400
+P 7950 1200
+F 0 "R190" V 7850 1200 50  0000 C CNN
+F 1 "470" V 8050 1200 50  0000 C CNN
+F 2 "" H 7950 1200 50  0001 C CNN
+F 3 "~" H 7950 1200 50  0001 C CNN
+	1    7950 1200
 	0    1    1    0
 $EndComp
@@
 $EndComp
 Wire Wire Line
-	2350 7600 2500 7600
+	2350 7600 2600 7600
 Wire Wire Line
 	1600 7700 1600 7750
@@
 Text Label 1250 7750 0    50   ~ 0
 SW2
-Wire Wire Line
-	2500 7600 2600 7600
-Connection ~ 2500 7600
+Connection ~ 2600 7600
 $Comp
 L power:+5V #PWR?
 U 1 1 5F0F560A
-P 2500 7600
-F 0 "#PWR?" H 2500 7450 50  0001 C CNN
-F 1 "+5V" H 2515 7773 50  0000 C CNN
-F 2 "" H 2500 7600 50  0001 C CNN
-F 3 "" H 2500 7600 50  0001 C CNN
-	1    2500 7600
+P 2600 7600
+F 0 "#PWR?" H 2600 7450 50  0001 C CNN
+F 1 "+5V" H 2615 7773 50  0000 C CNN
+F 2 "" H 2600 7600 50  0001 C CNN
+F 3 "" H 2600 7600 50  0001 C CNN
+	1    2600 7600
 	1    0    0    -1
 $EndComp
@@
 Wire Wire Line
 	2600 7600 2850 7600
-Connection ~ 2600 7600
 Wire Wire Line
 	2600 7650 2600 7600
@@
 	5150 5800 5350 5800
 Connection ~ 5350 5800
-Text Label 2450 1400 2    50   ~ 0
+Text Label 8450 1200 2    50   ~ 0
 J8-16
 Wire Wire Line
-	2050 1400 2450 1400
+	8050 1200 8450 1200
 $Comp
 L power:GNDREF #PWR?
@@
 Wire Wire Line
 	13200 8450 12800 8450
-Text Label 2450 1050 2    50   ~ 0
+Text Label 8450 850  2    50   ~ 0
 J8-4
-Text HLabel 1150 1050 0    50   Input ~ 0
+Text HLabel 7150 850  0    50   Input ~ 0
 3.5DIK
 Text HLabel 1200 2950 0    50   Input ~ 0
 Q3.H
-Text HLabel 1150 1400 0    50   Input ~ 0
+Text HLabel 7150 1200 0    50   Input ~ 0
 HDSEL.H
-Connection ~ 1700 1400
-Wire Wire Line
-	1850 1400 1700 1400
-Wire Wire Line
-	1150 1400 1700 1400
-Wire Wire Line
-	1700 1600 1700 1400
-Text Label 1700 1400 2    50   ~ 0
+Connection ~ 7700 1200
+Wire Wire Line
+	7850 1200 7700 1200
+Wire Wire Line
+	7150 1200 7700 1200
+Wire Wire Line
+	7700 1400 7700 1200
+Text Label 7700 1200 2    50   ~ 0
 HDSEL.H
 Wire Wire Line
-	2050 1050 2450 1050
+	8050 850  8450 850
 Text HLabel 950  5150 0    50   Input ~ 0
 RDY.H
