File: Apple/Apple IIGS/IIgs/ROM3 Schematic/Slots-7.sch (KiCad schematic (older format))
At the start: 22 parts, among them J1 Apple_II_Slot, J2 Apple_II_Slot, J3 Apple_II_Slot, J4 Apple_II_Slot, J5 Apple_II_Slot, J6 Apple_II_Slot, J7 Apple_II_Slot

Commit message: continued refinements
Connections:
- net MDBUS0: no longer UD5.11 (B8), UD5.12 (B7), UD5.13 (B6), UD5.14 (B5), UD5.15 (B4), UD5.16 (B3), UD5.17 (B2)
- new net MDBUS1: UD5.17 (B2)
- new net MDBUS2: UD5.16 (B3)
- new net MDBUS3: UD5.15 (B4)
- new net MDBUS4: UD5.14 (B5)
- new net MDBUS5: UD5.13 (B6)
- new net MDBUS6: UD5.12 (B7)
- new net MDBUS7: UD5.11 (B8)
Changed lines of the file:
@@
 $Descr A3 16535 11693
 encoding utf-8
-Sheet 7 10
+Sheet 1 1
 Title ""
 Date ""
@@
 Wire Wire Line
 	2000 6800 2000 6850
-Text Label 3450 8000 2    50   ~ 0
-MDBUS0
-Text Label 3450 8100 2    50   ~ 0
-MDBUS0
-Text Label 3450 8200 2    50   ~ 0
-MDBUS0
-Text Label 3450 8300 2    50   ~ 0
-MDBUS0
-Text Label 3450 8400 2    50   ~ 0
-MDBUS0
-Text Label 3450 8500 2    50   ~ 0
-MDBUS0
-Text Label 3450 8600 2    50   ~ 0
-MDBUS0
-Text Label 3450 8700 2    50   ~ 0
-MDBUS0
 Text Label 1850 7850 0    50   ~ 0
 MDIN-OUT
@@
 Text Notes 2500 7250 0    50   ~ 0
 C038-3F appears to be sound related\nhttps://www.kreativekorp.com/miscpages/a2info/iomemory.shtml
+Text Label 3450 8000 2    50   ~ 0
+MDBUS0
+Text Label 3450 8100 2    50   ~ 0
+MDBUS1
+Text Label 3450 8200 2    50   ~ 0
+MDBUS2
+Text Label 3450 8300 2    50   ~ 0
+MDBUS3
+Text Label 3450 8400 2    50   ~ 0
+MDBUS4
+Text Label 3450 8500 2    50   ~ 0
+MDBUS5
+Text Label 3450 8600 2    50   ~ 0
+MDBUS6
+Text Label 3450 8700 2    50   ~ 0
+MDBUS7
 $EndSCHEMATC
