File: Apple/Apple IIGS/IIgs/ROM3 Schematic/UG12-5.sch (KiCad schematic (older format))
At the start: 29 parts, among them J18 Apple Desk Top Bus, J21 Game-IO, J23 Edge Conn Burn-In, Q4 2N3904

Commit message: added more notes on keyboard page. refined some hierarchical labels.
Connections:
- net UI12-13: no longer RP1.7 (R6), UG12.4 (P20)
- net UI12-14: no longer RP1.8 (R7), UG12.3 (P21)
- net UI12-15: no longer RP1.9 (R8), UG12.2 (P22)
- net UI12-16: no longer RP1.10 (R9), UG12.1 (P23)
- net UI12-19 renamed UI12-STB
- new net UI12-SEL0: RP1.7 (R6), UG12.4 (P20)
- new net UI12-SEL1: RP1.8 (R7), UG12.3 (P21)
- new net UI12-SEL2: RP1.9 (R8), UG12.2 (P22)
- new net UI12-SEL3: RP1.10 (R9), UG12.1 (P23)
Other:
- note added: "UG12 is UI14 on 256K"
- note added: "UI14-35 and 34 are strange designations here. \nThey connected to the keyboard matrix on the \n256K IIgs (which 1MB doesn't have.)\n-35 is X1\n-34 is X2\n\nBut the rest of the matrix is missing."
- note added: "UL12 labels changed from schematic"
- moved on the sheet: JP?, R217
Changed lines of the file:
@@
 $EndDescr
-$Comp
-L IIgs-Schematic:M50741 UG12
-U 1 1 5BF205D4
-P 5400 3300
-F 0 "UG12" H 5550 4750 50  0000 C CNN
-F 1 "M50741" H 5600 4650 50  0000 C CNN
-F 2 "" H 4950 4700 50  0001 C CNN
-F 3 "" H 4950 4700 50  0001 C CNN
-	1    5400 3300
-	1    0    0    -1
-$EndComp
 $Comp
 L IIgs-Schematic:Game-IO J21
@@
 	9050 3000 8550 3000
 Text Label 8550 3000 0    50   ~ 0
-UI12-19
+UI12-STB
 Wire Wire Line
 	9050 2800 8550 2800
@@
 L IIgs-Schematic-rescue:M02-freetronics_schematic-IIgs-Schematic-rescue JP?
 U 1 1 5CB3AF62
-P 7600 3850
-F 0 "JP?" H 7578 3790 50  0000 L CNN
-F 1 "M02-freetronics_schematic" H 7578 3744 40  0001 L CNN
-F 2 "" H 7600 3850 60  0000 C CNN
-F 3 "" H 7600 3850 60  0000 C CNN
-	1    7600 3850
-	1    0    0    -1
-$EndComp
-Text Label 6850 3950 0    50   ~ 0
+P 7600 4950
+F 0 "JP?" H 7578 4890 50  0000 L CNN
+F 1 "M02-freetronics_schematic" H 7578 4844 40  0001 L CNN
+F 2 "" H 7600 4950 60  0000 C CNN
+F 3 "" H 7600 4950 60  0000 C CNN
+	1    7600 4950
+	1    0    0    -1
+$EndComp
+Text Label 6850 5050 0    50   ~ 0
 CP-CNTL
 Wire Wire Line
-	6850 3950 7250 3950
-Wire Wire Line
-	7300 3850 7250 3850
-Wire Wire Line
-	7250 3850 7250 3750
+	6850 5050 7250 5050
+Wire Wire Line
+	7300 4950 7250 4950
+Wire Wire Line
+	7250 4950 7250 4850
 $Comp
 L power:+5V #PWR?
 U 1 1 5CB3CD3A
-P 7250 3750
-F 0 "#PWR?" H 7250 3600 50  0001 C CNN
-F 1 "+5V" H 7265 3923 50  0000 C CNN
-F 2 "" H 7250 3750 50  0001 C CNN
-F 3 "" H 7250 3750 50  0001 C CNN
-	1    7250 3750
+P 7250 4850
+F 0 "#PWR?" H 7250 4700 50  0001 C CNN
+F 1 "+5V" H 7265 5023 50  0000 C CNN
+F 2 "" H 7250 4850 50  0001 C CNN
+F 3 "" H 7250 4850 50  0001 C CNN
+	1    7250 4850
 	1    0    0    -1
 $EndComp
@@
 L Device:R_Small R217
 U 1 1 5CB3CD82
-P 7250 4150
-F 0 "R217" H 7320 4196 50  0000 L CNN
-F 1 "4.7k" H 7320 4105 50  0000 L CNN
-F 2 "" V 7180 4150 50  0001 C CNN
-F 3 "~" H 7250 4150 50  0001 C CNN
-	1    7250 4150
-	1    0    0    -1
-$EndComp
-Connection ~ 7250 3950
-Wire Wire Line
-	7250 3950 7300 3950
+P 7250 5250
+F 0 "R217" H 7320 5296 50  0000 L CNN
+F 1 "4.7k" H 7320 5205 50  0000 L CNN
+F 2 "" V 7180 5250 50  0001 C CNN
+F 3 "~" H 7250 5250 50  0001 C CNN
+	1    7250 5250
+	1    0    0    -1
+$EndComp
+Connection ~ 7250 5050
+Wire Wire Line
+	7250 5050 7300 5050
 $Comp
 L power:GND #PWR?
 U 1 1 5CB3DD1A
-P 7250 4350
-F 0 "#PWR?" H 7250 4100 50  0001 C CNN
-F 1 "GND" H 7255 4177 50  0000 C CNN
-F 2 "" H 7250 4350 50  0001 C CNN
-F 3 "" H 7250 4350 50  0001 C CNN
-	1    7250 4350
+P 7250 5450
+F 0 "#PWR?" H 7250 5200 50  0001 C CNN
+F 1 "GND" H 7255 5277 50  0000 C CNN
+F 2 "" H 7250 5450 50  0001 C CNN
+F 3 "" H 7250 5450 50  0001 C CNN
+	1    7250 5450
 	1    0    0    -1
 $EndComp
@@
 	3450 2850 3850 2850
 Text Label 3850 2850 2    50   ~ 0
-UI12-19
+UI12-STB
 Wire Wire Line
 	6850 1900 6800 1900
@@
 	0    -1   -1   0
 $EndComp
-Text Label 7650 1400 2    50   ~ 0
-UI12-13
-Text Label 7650 1300 2    50   ~ 0
-UI12-14
-Text Label 7650 1200 2    50   ~ 0
-UI12-15
-Wire Wire Line
-	7650 1400 7250 1400
-Wire Wire Line
-	7250 1300 7650 1300
-Wire Wire Line
-	7650 1200 7250 1200
-Wire Wire Line
-	7250 1100 7650 1100
+Text Label 7750 1400 2    50   ~ 0
+UI12-SEL0
+Text Label 7750 1300 2    50   ~ 0
+UI12-SEL1
+Text Label 7750 1200 2    50   ~ 0
+UI12-SEL2
+Wire Wire Line
+	7750 1400 7250 1400
+Wire Wire Line
+	7250 1300 7750 1300
+Wire Wire Line
+	7750 1200 7250 1200
+Wire Wire Line
+	7250 1100 7750 1100
 Text Label 7650 1600 2    50   ~ 0
 UI14-34
@@
 L2-8
 Text Label 4250 2650 0    50   ~ 0
-UI12-14
+UI12-SEL1
 Text Label 4250 2550 0    50   ~ 0
-UI12-15
+UI12-SEL2
 Text Label 4250 2450 0    50   ~ 0
-UI12-16
+UI12-SEL3
 Text Label 4250 2350 0    50   ~ 0
-UI12-19
+UI12-STB
 Wire Wire Line
 	4250 2650 4750 2650
@@
 Wire Wire Line
 	4750 2350 4250 2350
-Text Label 7650 1100 2    50   ~ 0
-UI12-16
+Text Label 7750 1100 2    50   ~ 0
+UI12-SEL3
 Text Label 4250 2750 0    50   ~ 0
-UI12-13
+UI12-SEL0
 Wire Wire Line
 	4250 2750 4750 2750
@@
 	6950 3000 6950 3050
 Wire Wire Line
-	7250 3950 7250 4050
-Wire Wire Line
-	7250 4250 7250 4350
+	7250 5050 7250 5150
+Wire Wire Line
+	7250 5350 7250 5450
 Wire Wire Line
 	3950 6650 3950 7050
@@
 Wire Wire Line
 	8600 1900 9050 1900
-Text Notes 10100 3850 2    50   ~ 0
+Text Notes 10100 3850 2    39   ~ 0
 Does KEYGLU also do matrix decoding?!\n(For the Apple IIe Keyboard connector)
 Text HLabel 8600 4950 0    50   Input ~ 0
@@
 Wire Wire Line
 	4550 4050 4750 4050
+$Comp
+L IIgs-Schematic:M50741 UG12
+U 1 1 5BF205D4
+P 5400 3300
+F 0 "UG12" H 5550 4750 50  0000 C CNN
+F 1 "M50741" H 5600 4650 50  0000 C CNN
+F 2 "" H 4950 4700 50  0001 C CNN
+F 3 "" H 4950 4700 50  0001 C CNN
+	1    5400 3300
+	1    0    0    -1
+$EndComp
+Text Notes 4900 1400 0    50   ~ 0
+UG12 is UI14 on 256K
+Text Notes 2550 2500 0    50   ~ 0
+UL12 labels changed from schematic
+Text Notes 6700 3900 0    39   ~ 0
+UI14-35 and 34 are strange designations here. \nThey connected to the keyboard matrix on the \n256K IIgs (which 1MB doesn't have.)\n-35 is X1\n-34 is X2\n\nBut the rest of the matrix is missing.
 $EndSCHEMATC

Commit message: More label style changes
Other:
- note removed: "Does KEYGLU also do matrix decoding?!\n(For the Apple IIe Keyboard connector)"
Changed lines of the file:
@@
 Wire Wire Line
 	8600 1900 9050 1900
-Text Notes 10100 3850 2    39   ~ 0
-Does KEYGLU also do matrix decoding?!\n(For the Apple IIe Keyboard connector)
 Text HLabel 8600 4950 0    50   Input ~ 0
 SW0-OAPL

Commit message: continued fixes while working on golden delicious project
Connections:
- net AN0: now also J21.15; no longer J21.16
- net AN1: now also J21.14; no longer J21.15
- net AN2: now also J21.13; no longer J21.14
- net AN3: now also J21.12; no longer J21.13
- net PDL1: no longer J21.12
- no-connect marks 0 -> 1
Other:
- moved on the sheet: J21, R117
Changed lines of the file:
@@
 L IIgs-Schematic:Game-IO J21
 U 1 1 5BF2066B
-P 1650 6800
-F 0 "J21" H 1650 7250 50  0000 C CNN
-F 1 "Game-IO" H 1650 6350 50  0000 C CNN
-F 2 "" H 1650 7300 50  0001 C CNN
-F 3 "" H 1650 7300 50  0001 C CNN
-	1    1650 6800
+P 2000 6800
+F 0 "J21" H 2000 7250 50  0000 C CNN
+F 1 "Game-IO" H 2000 6350 50  0000 C CNN
+F 2 "" H 2000 7300 50  0001 C CNN
+F 3 "" H 2000 7300 50  0001 C CNN
+	1    2000 6800
 	1    0    0    -1
 $EndComp
@@
 Text Label 4250 3850 0    50   ~ 0
 VBL.L
-Text Label 2250 7050 2    50   ~ 0
+Text Label 2600 7050 2    50   ~ 0
 PDL1
 Wire Wire Line
-	2250 7050 1950 7050
-Text Label 2250 6950 2    50   ~ 0
+	2600 7050 2300 7050
+Text Label 2600 6950 2    50   ~ 0
 PDL3
 Wire Wire Line
-	2250 6950 1950 6950
-Text Label 2250 6850 2    50   ~ 0
-PDL1
-Wire Wire Line
-	2250 6850 1950 6850
-Text Label 2250 6750 2    50   ~ 0
+	2600 6950 2300 6950
+Text Label 2600 6850 2    50   ~ 0
 AN3
 Wire Wire Line
-	2250 6750 1950 6750
-Text Label 2250 6650 2    50   ~ 0
+	2600 6850 2300 6850
+Text Label 2600 6750 2    50   ~ 0
 AN2
 Wire Wire Line
-	2250 6650 1950 6650
-Text Label 2250 6550 2    50   ~ 0
+	2600 6750 2300 6750
+Text Label 2600 6650 2    50   ~ 0
 AN1
 Wire Wire Line
-	2250 6550 1950 6550
-Text Label 2250 6450 2    50   ~ 0
+	2600 6650 2300 6650
+Text Label 2600 6550 2    50   ~ 0
 AN0
 Wire Wire Line
-	2250 6450 1950 6450
-Text Label 2250 7150 2    50   ~ 0
+	2600 6550 2300 6550
+Text Label 2600 7150 2    50   ~ 0
 SW3
 Wire Wire Line
-	2250 7150 1950 7150
-Wire Wire Line
-	1350 6450 1250 6450
-Wire Wire Line
-	1250 6450 1250 6400
+	2600 7150 2300 7150
+Wire Wire Line
+	1700 6450 1600 6450
+Wire Wire Line
+	1600 6450 1600 6400
 $Comp
 L power:+5V #PWR?
 U 1 1 5CFE6032
-P 1250 6400
-F 0 "#PWR?" H 1250 6250 50  0001 C CNN
-F 1 "+5V" H 1265 6573 50  0000 C CNN
-F 2 "" H 1250 6400 50  0001 C CNN
-F 3 "" H 1250 6400 50  0001 C CNN
-	1    1250 6400
-	1    0    0    -1
-$EndComp
-Text Label 850  6550 0    50   ~ 0
+P 1600 6400
+F 0 "#PWR?" H 1600 6250 50  0001 C CNN
+F 1 "+5V" H 1615 6573 50  0000 C CNN
+F 2 "" H 1600 6400 50  0001 C CNN
+F 3 "" H 1600 6400 50  0001 C CNN
+	1    1600 6400
+	1    0    0    -1
+$EndComp
+Text Label 1200 6550 0    50   ~ 0
 SW0-OAPL
-Text Label 850  6650 0    50   ~ 0
+Text Label 1200 6650 0    50   ~ 0
 SW1-CAPL
 Wire Wire Line
-	850  6550 1350 6550
-Wire Wire Line
-	850  6650 1350 6650
+	1200 6550 1700 6550
+Wire Wire Line
+	1200 6650 1700 6650
 $Comp
 L Device:R_Small R117
 U 1 1 5D009004
-P 950 6900
-F 0 "R117" V 850 6900 50  0000 C CNN
-F 1 "4.7K" V 1050 6900 50  0000 C CNN
-F 2 "" V 880 6900 50  0001 C CNN
-F 3 "~" H 950 6900 50  0001 C CNN
-	1    950  6900
+P 1300 6900
+F 0 "R117" V 1200 6900 50  0000 C CNN
+F 1 "4.7K" V 1400 6900 50  0000 C CNN
+F 2 "" V 1230 6900 50  0001 C CNN
+F 3 "~" H 1300 6900 50  0001 C CNN
+	1    1300 6900
 	0    1    1    0
 $EndComp
 Wire Wire Line
-	1150 6900 1150 6850
-Wire Wire Line
-	1150 6850 1350 6850
+	1500 6900 1500 6850
+Wire Wire Line
+	1500 6850 1700 6850
 $Comp
 L power:+5V #PWR?
 U 1 1 5D02D882
-P 750 6900
-F 0 "#PWR?" H 750 6750 50  0001 C CNN
-F 1 "+5V" V 765 7028 50  0000 L CNN
-F 2 "" H 750 6900 50  0001 C CNN
-F 3 "" H 750 6900 50  0001 C CNN
-	1    750  6900
+P 1100 6900
+F 0 "#PWR?" H 1100 6750 50  0001 C CNN
+F 1 "+5V" V 1115 7028 50  0000 L CNN
+F 2 "" H 1100 6900 50  0001 C CNN
+F 3 "" H 1100 6900 50  0001 C CNN
+	1    1100 6900
 	0    -1   -1   0
 $EndComp
-Text Label 1150 6850 0    50   ~ 0
+Text Label 1500 6850 0    50   ~ 0
 STB.L
 Wire Wire Line
-	1350 6950 1150 6950
-Wire Wire Line
-	1150 7150 850  7150
-Wire Wire Line
-	1150 6950 1150 7150
-Text Label 850  7150 0    50   ~ 0
+	1700 6950 1500 6950
+Wire Wire Line
+	1500 7150 1200 7150
+Wire Wire Line
+	1500 6950 1500 7150
+Text Label 1200 7150 0    50   ~ 0
 PDL0
 Wire Wire Line
-	1350 7050 1200 7050
-Wire Wire Line
-	1200 7050 1200 7250
-Wire Wire Line
-	1200 7250 850  7250
-Text Label 850  7250 0    50   ~ 0
+	1700 7050 1550 7050
+Wire Wire Line
+	1550 7050 1550 7250
+Wire Wire Line
+	1550 7250 1200 7250
+Text Label 1200 7250 0    50   ~ 0
 PDL2
 Wire Wire Line
-	850  6750 1350 6750
-Text Label 850  6750 0    50   ~ 0
+	1200 6750 1700 6750
+Text Label 1200 6750 0    50   ~ 0
 SW2
 Wire Wire Line
-	1350 7150 1300 7150
-Wire Wire Line
-	1300 7150 1300 7250
+	1700 7150 1650 7150
+Wire Wire Line
+	1650 7150 1650 7250
 $Comp
 L power:GND #PWR?
 U 1 1 5D0A3210
-P 1300 7250
-F 0 "#PWR?" H 1300 7000 50  0001 C CNN
-F 1 "GND" H 1305 7077 50  0000 C CNN
-F 2 "" H 1300 7250 50  0001 C CNN
-F 3 "" H 1300 7250 50  0001 C CNN
-	1    1300 7250
+P 1650 7250
+F 0 "#PWR?" H 1650 7000 50  0001 C CNN
+F 1 "GND" H 1655 7077 50  0000 C CNN
+F 2 "" H 1650 7250 50  0001 C CNN
+F 3 "" H 1650 7250 50  0001 C CNN
+	1    1650 7250
 	1    0    0    -1
 $EndComp
@@
 	6600 7200 6600 7300
 Wire Wire Line
-	750  6900 850  6900
-Wire Wire Line
-	1050 6900 1150 6900
+	1100 6900 1200 6900
+Wire Wire Line
+	1400 6900 1500 6900
 Text HLabel 4350 4250 0    39   Input ~ 0
 CREF.H
@@
 Text HLabel 8600 4950 0    50   Input ~ 0
 SW0-OAPL
-Text HLabel 7350 2650 2    50   Input ~ 0
-SW1-OAPL
-Wire Wire Line
-	7350 2650 7250 2650
-Connection ~ 7250 2650
 Text Notes 4900 5450 0    50   ~ 0
 Mitsubishi 740 Microcontroller\n(6502 based)\nfor ADB
@@
 Text Notes 6700 3900 0    39   ~ 0
 UI14-35 and 34 are strange designations here. \nThey connected to the keyboard matrix on the \n256K IIgs (which 1MB doesn't have.)\n-35 is X1\n-34 is X2\n\nBut the rest of the matrix is missing.
+Text HLabel 1200 6650 0    50   Input ~ 0
+SW1-OAPL
+Text HLabel 1200 6550 0    50   Input ~ 0
+SW0-OAPL
+NoConn ~ 2300 6450
 $EndSCHEMATC
